Commit message: Fix assembly visualization for OrcaHand-equipped OpenArm

File: assembly_description/urdf/assembly.urdf (robot description, URDF)
Before this commit: robot openarm_orca_stack, 0 links, 2 joints
Joints:
- joint left_hand_joint: child left_palm -> left_tower
- joint right_hand_joint: child right_palm -> right_tower

File: orcahand_description/models/urdf/orcahand_left.urdf (robot description, URDF)
Before this commit: robot orcahand_left, 42 links, 41 joints
Links:
- removed link world
- removed link world2left_tower_fixed_jointbody
Joints:
- removed joint world2left_tower_fixed
- removed joint world2left_tower_fixed_offset

File: orcahand_description/models/urdf/orcahand_left_extended.urdf (robot description, URDF)
Before this commit: robot orcahand_left_extended, 42 links, 41 joints
Links:
- removed link world
- removed link world2left_tower_fixed_jointbody
Joints:
- removed joint world2left_tower_fixed
- removed joint world2left_tower_fixed_offset

File: orcahand_description/models/urdf/orcahand_right.urdf (robot description, URDF)
Before this commit: robot orcahand_right, 42 links, 41 joints
Links:
- removed link world
- removed link world2right_tower_fixed_jointbody
Joints:
- removed joint world2right_tower_fixed
- removed joint world2right_tower_fixed_offset

File: orcahand_description/models/urdf/orcahand_right_extended.urdf (robot description, URDF)
Before this commit: robot orcahand_right_extended, 42 links, 41 joints
Links:
- removed link world
- removed link world2right_tower_fixed_jointbody
Joints:
- removed joint world2right_tower_fixed
- removed joint world2right_tower_fixed_offset

Commit message: Fix OpenArm assembly integration for ORCA hands

File: assembly_description/urdf/assembly.urdf (robot description, URDF)
Before this commit: robot openarm_orca_stack, 0 links, 2 joints
Joints:
- joint left_hand_joint: child left_palm -> left_tower
- joint right_hand_joint: child right_palm -> right_tower

Commit message: Remove unused base link attachment parameter

File: assembly_description/urdf/assembly.urdf (robot description, URDF)
Before this commit: robot openarm_orca_stack, 0 links, 2 joints
Links:
- added link $(arg parent)
Joints:
- added joint openarm_world_joint: type fixed, parent $(arg parent), child openarm_body_link0, origin xyz=$(arg xyz) rpy=$(arg rpy)
- joint left_hand_joint: child left_palm -> left_tower
- joint right_hand_joint: child right_palm -> right_tower

Commit message: Fix duplicate world roots in modular assembly

File: assembly_description/urdf/assembly.urdf (robot description, URDF)
Before this commit: robot openarm_orca_stack, 0 links, 2 joints
Links:
- added link ${root_link}

File: openarm_description/urdf/body/openarm_body.xacro (robot description, xacro)
@@ -8,4 +8,5 @@
               description_pkg:='openarm_description'
               connected_to:='world'
+              create_parent_link:=true
               xyz:='0 0 0'
               rpy:='0 0 0'
@@ -16,5 +17,7 @@
     <xacro:property name="prefix" value="${'' if no_prefix else 'openarm_' + 'body_'}" />
     <xacro:unless value="${not connected_to}">
-    <link name="${connected_to}" />
+    <xacro:if value="${create_parent_link}">
+      <link name="${connected_to}" />
+    </xacro:if>
     <joint name="${prefix}${connected_to}_joint" type="fixed">
     <parent link="${connected_to}" />

File: openarm_description/urdf/robot/openarm_robot.xacro (robot description, xacro)
@@ -27,4 +27,5 @@
             arm_connected_to='base'
             body_connected_to='world'
+            body_create_parent_link:='true'
             bimanual:=false
             right_arm_base_xyz='0 0 0'
@@ -59,4 +60,5 @@
         description_pkg="openarm_description"
         connected_to="${body_connected_to}"
+        create_parent_link="${body_create_parent_link}"
         xyz="${xyz}"
         rpy="${rpy}"
